File: Frienduino.sch (EAGLE design)
At the start: 31 parts, among them IC1 ATMEGA328, IC2 PIC16F1454, Q2 16MHz

Commit message: changed resistors to 7mm raster
Parts:
- R1, R4, R5, R6, R7, R8, R9: device rcl:R-EU_0204/5 -> resistor:R-EU_0204/7
Changed lines of the file:
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@@
 <part name="P+1" library="supply1" deviceset="+5V" device=""/>
 <part name="GND1" library="supply1" deviceset="GND" device=""/>
-<part name="R1" library="rcl" deviceset="R-EU_" device="0204/5" value="10k"/>
+<part name="R1" library="resistor" deviceset="R-EU_" device="0204/7" value="10k"/>
 <part name="P+2" library="supply1" deviceset="+5V" device=""/>
 <part name="C1" library="rcl" deviceset="C-EU" device="050-025X075" value="100n"/>
@@
 <part name="S1" library="switch-omron" deviceset="10-XX" device=""/>
 <part name="GND12" library="supply1" deviceset="GND" device=""/>
-<part name="R7" library="rcl" deviceset="R-EU_" device="0204/5" value="1k"/>
+<part name="R7" library="resistor" deviceset="R-EU_" device="0204/7" value="1k"/>
 <part name="GND8" library="supply1" deviceset="GND" device=""/>
 <part name="PWR" library="led" deviceset="LED" device="3MM"/>
 <part name="GND14" library="supply1" deviceset="GND" device=""/>
-<part name="R6" library="rcl" deviceset="R-EU_" device="0204/5" value="1k"/>
+<part name="R6" library="resistor" deviceset="R-EU_" device="0204/7" value="1k"/>
 <part name="P+5" library="supply1" deviceset="+5V" device=""/>
 <part name="RX" library="led" deviceset="LED" device="3MM"/>
 <part name="TX" library="led" deviceset="LED" device="3MM"/>
-<part name="R4" library="rcl" deviceset="R-EU_" device="0204/5" value="1k"/>
-<part name="R5" library="rcl" deviceset="R-EU_" device="0204/5" value="1k"/>
-<part name="R8" library="rcl" deviceset="R-EU_" device="0204/5" value="1k"/>
-<part name="R9" library="rcl" deviceset="R-EU_" device="0204/5" value="1k"/>
+<part name="R4" library="resistor" deviceset="R-EU_" device="0204/7" value="1k"/>
+<part name="R5" library="resistor" deviceset="R-EU_" device="0204/7" value="1k"/>
+<part name="R8" library="resistor" deviceset="R-EU_" device="0204/7" value="1k"/>
+<part name="R9" library="resistor" deviceset="R-EU_" device="0204/7" value="1k"/>
 <part name="Q2" library="crystal" deviceset="CRYTAL" device="HC49S" value="16MHz"/>
 <part name="X4" library="SmartPrj" deviceset="PN61729" device=""/>

Commit message: prepared board for manufacture and added gergers
Parts:
- ICSP: value (none) -> ISP
- SV1: value (none) -> PIC ICSP
Changed lines of the file:
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@@
 <layer number="51" name="tDocu" color="15" fill="1" visible="no" active="no"/>
 <layer number="52" name="bDocu" color="7" fill="1" visible="no" active="no"/>
+<layer number="53" name="tGND_GNDA" color="7" fill="9" visible="no" active="no"/>
+<layer number="54" name="bGND_GNDA" color="1" fill="9" visible="no" active="no"/>
+<layer number="56" name="wert" color="7" fill="1" visible="no" active="no"/>
 <layer number="91" name="Nets" color="2" fill="1" visible="yes" active="yes"/>
 <layer number="92" name="Busses" color="1" fill="1" visible="yes" active="yes"/>
@@
 <layer number="97" name="Info" color="7" fill="1" visible="yes" active="yes"/>
 <layer number="98" name="Guide" color="6" fill="1" visible="yes" active="yes"/>
+<layer number="100" name="Muster" color="7" fill="1" visible="no" active="no"/>
+<layer number="101" name="Patch_Top" color="12" fill="4" visible="yes" active="yes"/>
+<layer number="102" name="Vscore" color="7" fill="1" visible="yes" active="yes"/>
+<layer number="103" name="tMap" color="7" fill="1" visible="yes" active="yes"/>
+<layer number="104" name="Name" color="7" fill="1" visible="yes" active="yes"/>
+<layer number="105" name="tPlate" color="7" fill="1" visible="yes" active="yes"/>
+<layer number="106" name="bPlate" color="7" fill="1" visible="yes" active="yes"/>
+<layer number="107" name="Crop" color="7" fill="1" visible="yes" active="yes"/>
+<layer number="116" name="Patch_BOT" color="9" fill="4" visible="yes" active="yes"/>
+<layer number="121" name="_tsilk" color="7" fill="1" visible="yes" active="yes"/>
+<layer number="122" name="_bsilk" color="7" fill="1" visible="yes" active="yes"/>
+<layer number="125" name="_tNames" color="7" fill="1" visible="yes" active="yes"/>
+<layer number="144" name="Drill_legend" color="7" fill="1" visible="yes" active="yes"/>
+<layer number="151" name="HeatSink" color="7" fill="1" visible="yes" active="yes"/>
 <layer number="200" name="200bmp" color="1" fill="10" visible="no" active="no"/>
+<layer number="201" name="201bmp" color="2" fill="10" visible="yes" active="yes"/>
+<layer number="202" name="202bmp" color="3" fill="10" visible="yes" active="yes"/>
+<layer number="203" name="203bmp" color="4" fill="10" visible="yes" active="yes"/>
+<layer number="204" name="204bmp" color="5" fill="10" visible="yes" active="yes"/>
+<layer number="205" name="205bmp" color="6" fill="10" visible="yes" active="yes"/>
+<layer number="206" name="206bmp" color="7" fill="10" visible="yes" active="yes"/>
+<layer number="207" name="207bmp" color="8" fill="10" visible="yes" active="yes"/>
+<layer number="208" name="208bmp" color="9" fill="10" visible="yes" active="yes"/>
+<layer number="209" name="209bmp" color="7" fill="1" visible="yes" active="yes"/>
+<layer number="210" name="210bmp" color="7" fill="1" visible="yes" active="yes"/>
+<layer number="211" name="211bmp" color="7" fill="1" visible="yes" active="yes"/>
+<layer number="212" name="212bmp" color="7" fill="1" visible="yes" active="yes"/>
+<layer number="213" name="213bmp" color="7" fill="1" visible="yes" active="yes"/>
+<layer number="214" name="214bmp" color="7" fill="1" visible="yes" active="yes"/>
+<layer number="215" name="215bmp" color="7" fill="1" visible="yes" active="yes"/>
+<layer number="216" name="216bmp" color="7" fill="1" visible="yes" active="yes"/>
 <layer number="250" name="Descript" color="3" fill="1" visible="no" active="no"/>
 <layer number="251" name="SMDround" color="12" fill="11" visible="no" active="no"/>
+<layer number="254" name="cooling" color="7" fill="1" visible="yes" active="yes"/>
 </layers>
 <schematic>
@@
 <parts>
 <part name="IC1" library="atmel" deviceset="AT90S4433" device="P" value="ATMEGA328"/>
-<part name="ICSP" library="pinhead" deviceset="PINHD-2X3" device=""/>
+<part name="ICSP" library="pinhead" deviceset="PINHD-2X3" device="" value="ISP"/>
 <part name="P+1" library="supply1" deviceset="+5V" device=""/>
 <part name="GND1" library="supply1" deviceset="GND" device=""/>
@@
 <part name="GND6" library="supply1" deviceset="GND" device=""/>
 <part name="C4" library="rcl" deviceset="C-EU" device="050-025X075" value="470n"/>
-<part name="SV1" library="con-lstb" deviceset="MA05-1" device=""/>
+<part name="SV1" library="con-lstb" deviceset="MA05-1" device="" value="PIC ICSP"/>
 <part name="D1" library="diode" deviceset="SCHOTTKY-DIODE" device="DO35-7" value="BAT 47"/>
 </parts>
